File: hardware/notifier-v1/display.kicad_sch (KiCad schematic)
At the start: 2 parts, among them J2 GC9A01 DISPLAY

Commit message: Layout A: USB-C on the back edge, corner mounts, no buttons, JLC fab data
- J2 display socket mirrored (1 RST 2 CS 3 DC 4 SDA 5 SCL 6 GND 7 VCC),
  face at the right edge
- USB-C J1 on the left edge (enclosure back), ESD/CC/fuse beside it,
  hand-drawn 0.27/0.15 pair (~91 ohm diff, tools/impedance.py), only
  GND under the shell (DRC rule area)
- SW1-SW3/R6/BTN removed; 1.5 mm debug pads TX RX 3V3 EN GND IO0;
  firmware DESK_BTN = -1 on notifier-v1
- Four M2 corner holes with keepouts; sensor island grown to 14.8 mm
  with H3 in its corner, re-hand-routed (BME688/SHT40 8.9 mm apart)
- I2C >= 1.6 mm from USB on the same layer; vias >= 0.15 mm from
  same-net SMD pads (rule), hand vias >= 0.2 mm
- Silk "v1 ${GIT_SHA}" resolved at fab export; JLC order-number mark
- Fab: Protel gerbers without X2, PTH/NPTH split, JLC BOM/CPL, CPL
  rotation fixes (U4 +90, U5 +270); pipeline --fab-only on a clean
  commit; route retry until the gate passes
- ORDER.md: stackup JLC04161H-7628, rails left/right, preview checklist,
  bring-up without buttons; PLAN.md enclosure notes

Co-Authored-By: Claude Opus 5.5 <noreply@anthropic.com>
Connections:
- net GND: now also J2.6 (Pin_6); no longer J2.2 (Pin_2)
- net LCD_CS: now also J2.2 (Pin_2); no longer J2.6 (Pin_6)
- net LCD_DC: now also J2.3 (Pin_3); no longer J2.5 (Pin_5)
- net LCD_RST: now also J2.1 (Pin_1); no longer J2.7 (Pin_7)
- net LCD_SCLK: now also J2.5 (Pin_5); no longer J2.3 (Pin_3)
- net LCD_VCC: now also J2.7 (Pin_7); no longer J2.1 (Pin_1)
Other:
- note added: "Notes - JP1: 1-2 bridged = LCD_VCC from 3V3 (default, 3.3 V modules). For 5 V modules cut the 1-2 bridge and bridge 2-3 (VBUS). - J2 pin order (mirrored for the right-edge socket): RST, CS, DC, SDA, SCL, GND, VCC (no MISO, no backlight pin). - Display plugs in from the side; its face sits past the board edge."
- note removed: "Notes - JP1: 1-2 bridged = LCD_VCC from 3V3 (default, 3.3 V modules). For 5 V modules cut the 1-2 bridge and bridge 2-3 (VBUS). - J2 pin order = module header: VCC, GND, SCL, SDA, DC, CS, RST (no MISO, no backlight pin). - Display plugs in from the side; its face sits past the board edge."
